File: instrumentation amplifier.kicad_pcb (KiCad board)
At the start: 2 copper layers, 22.9 x 22.2 mm, 13 parts, among them J1 Conn_02x02_Odd_Even, J2 Conn_02x01, J3 Conn_02x01, U1 TL074

Commit message: release v1
Parts:
- R7: value R -> 100
- moved R2 61.4 mm to (141.0, 144.4), turned to 90 degrees
- moved R4 61.4 mm to (138.7, 144.4)
- moved U1 61.4 mm to (135.9, 130.2)
- moved R1 61.4 mm to (141.0, 131.2)
- moved R3 61.4 mm to (138.7, 131.2)
- moved R5 61.4 mm to (132.7, 141.9)
- moved R6 61.4 mm to (138.7, 137.8)
- moved R7 61.4 mm to (141.0, 137.8)
- moved J2 61.4 mm to (132.1, 146.7)
- moved R9 61.4 mm to (132.1, 129.9)
- moved J3 61.4 mm to (132.1, 137.2)
- moved R8 61.4 mm to (132.1, 141.9)
- moved J1 57.0 mm to (147.3, 135.3), turned to 0 degrees
Connections:
- R2 pad 1: Net-(U1C--) -> Net-(R2-Pad1)
- R2 pad 2: Net-(R2-Pad2) -> Net-(U1C--)
- R4 pad 1: Net-(R2-Pad2) -> Net-(R2-Pad1)
- U1 pad 10: Net-(J1-Pin_1) -> Net-(J1-Pin_3)
- U1 pad 12: Net-(J1-Pin_3) -> Net-(J1-Pin_1)
- U1 pad 8: Net-(R2-Pad2) -> Net-(R2-Pad1)
Routing:
- net Net-(R2-Pad2): track 5.06 -> 0.00 mm
- net Net-(R2-Pad1): track 0.00 -> 5.06 mm
